File: NFC/NFC.kicad_pcb (KiCad board)
At the start: 2 copper layers, 3 parts, among them U1 NFC IC

Commit message: Initial dump to fix old issues and resume working on this project
Parts:
- added ANT1: PCB Antenna, NFC_Antenna:Class4_48x25mm_5T, F.Cu at (66.0, 66.7)
- moved C2 26.5 mm to (74.0, 73.0), turned to 180 degrees
- moved U1 25.6 mm to (74.0, 67.0)
- moved C1 22.5 mm to (80.5, 67.0)
Routing:
- net Net-(U1-LB): track 0.00 -> 40.3 mm
- net GND: track 0.00 -> 25.0 mm
- net Net-(U1-LA): track 0.00 -> 17.4 mm
- net Net-(U1-VCC): track 0.00 -> 4.28 mm
Other:
- board outline added: 85.6 x 54 mm
