File: NFC/NFC.kicad_sch (KiCad schematic)
At the start: 4 parts, among them U1 NFC IC

Commit message: Initial dump to fix old issues and resume working on this project
Parts:
- ANT1: footprint (none) -> NFC_Antenna:Class4_48x25mm_5T
Changed lines of the file:
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@@
 		(exclude_from_sim no)
 		(in_bom yes)
-		(on_board no)
+		(on_board yes)
 		(in_pos_files yes)
 		(dnp no)
@@
 			)
 		)
-		(property "Footprint" ""
+		(property "Footprint" "NFC_Antenna:Class4_48x25mm_5T"
 			(at 149.86 78.74 0)
 			(hide yes)
