File: schematic/project/project.kicad_pcb (KiCad board)
At the start: 2 copper layers, 85.6 x 54 mm, 11 parts, among them U1 NT3H2111W0FHKH

Commit message: Finalized card's design
Parts:
- LED1: value LED -> LED_Yellow; footprint LED_SMD:LED_0805_2012Metric -> LED_SMD:LED_0603_1608Metric; moved to B.Cu
- R1: value 47Ω -> 1 kΩ
- U1: value NT3H2111W0FHKH -> NT3H2111W0FTTJ; footprint NT3H2111W0FHKH:QFN8P50_160X160X50L40X20N -> Package_SO:TSSOP-8_3x3mm_P0.65mm
- moved LED1 12.2 mm to (161.0, 89.3), turned to -90 degrees
- moved R1 6.83 mm to (162.5, 79.0), turned to 180 degrees
- moved C1 3.47 mm to (158.9, 80.0), turned to 180 degrees
- moved G*** 1.82 mm to (127.2, 64.0)
- moved U1 1.67 mm to (157.8, 77.0)
Connections:
- net Net-(LED1-K) renamed GND
- C1 pad 1: Net-(U1-VCC) -> Net-(U1-VOUT)
- R1 pad 2: Net-(U1-VCC) -> Net-(U1-VOUT)
- U1 pad 6: Net-(U1-VCC) -> unconnected-(U1-VCC-Pad6)
- U1 pad 7: Net-(U1-VCC) -> Net-(U1-VOUT)
Routing:
- net Net-(U1-VCC): track 13.9 -> 0.00 mm
- net Net-(LED1-A): track 2.02 -> 13.1 mm, vias 0 -> 1
- net GND: track 8.20 -> 17.9 mm, vias 0 -> 1
- net Net-(U1-VOUT): track 0.00 -> 6.02 mm
- net Net-(U1-LA): track 7.18 -> 3.39 mm

Commit message: Added production files
Parts:
- LED1: value LED_Yellow -> APT1608SYCK/J3-PRV
- U1: value NT3H2111W0FTTJ -> NT3H2211W0FTTJ
Changed lines of the file:
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@@
 			)
 		)
-		(property "Value" "NT3H2111W0FTTJ"
+		(property "Value" "NT3H2211W0FTTJ"
 			(at 0 2.55 0)
 			(layer "F.Fab")
@@
 			)
 		)
+		(property "LCSC Part #" "C2654822"
+			(at 0 0 0)
+			(unlocked yes)
+			(layer "F.Fab")
+			(hide yes)
+			(effects
+				(font
+					(size 1 1)
+					(thickness 0.15)
+				)
+			)
+		)
 		(sheetname "/")
 		(sheetfile "project.kicad_sch")
+		(units
+			(unit
+				(name "A")
+				(pins "6" "5" "4" "3" "1" "8" "7" "2")
+			)
+		)
 		(clearance 0.2)
 		(attr smd)
@@
 			)
 		)
+		(property "LCSC Part #" "C17513"
+			(at 0 0 180)
+			(unlocked yes)
+			(layer "F.Fab")
+			(hide yes)
+			(effects
+				(font
+					(size 1 1)
+					(thickness 0.15)
+				)
+			)
+		)
 		(property ki_fp_filters "R_*")
 		(sheetname "/")
@@
 			)
 		)
-		(property "Datasheet" ""
+		(property "Datasheet" "file:///Users/maciej/Desktop/NT3H2111/docs/AN11276.pdf"
 			(at 0 0 0)
 			(layer "F.Fab")
@@
 			)
 		)
+		(property "LCSC Part #" "C520076"
+			(at 0 0 180)
+			(unlocked yes)
+			(layer "F.Fab")
+			(hide yes)
+			(effects
+				(font
+					(size 1 1)
+					(thickness 0.15)
+				)
+			)
+		)
 		(property ki_fp_filters "C_*")
 		(sheetname "/")
@@
 			)
 		)
-		(property "Value" "LED_Yellow"
+		(property "Value" "APT1608SYCK/J3-PRV"
 			(at 0 -1.43 90)
 			(layer "B.Fab")
@@
 			)
 		)
+		(property "LCSC Part #" "C5440241"
+			(at 0 0 270)
+			(unlocked yes)
+			(layer "B.Fab")
+			(hide yes)
+			(effects
+				(font
+					(size 1 1)
+					(thickness 0.15)
+				)
+				(justify mirror)
+			)
+		)
 		(property ki_fp_filters "LED* LED_SMD:* LED_THT:*")
 		(sheetname "/")
 		(sheetfile "project.kicad_sch")
+		(units
+			(unit
+				(name "A")
+				(pins "1" "2")
+			)
+		)
 		(attr smd)
 		(duplicate_pad_numbers_are_jumpers no)
