File: schematic/project/project.kicad_sch (KiCad schematic)
At the start: 4 parts, among them U1 NFC IC

Commit message: ??
After not realizing for nearly two weeks I finally committed proper workfiles with updated progress on the PCB of the card
Parts:
- removed C2: DNP, Capacitor_SMD:C_0805_2012Metric, symbol Device:C
- removed U1: NFC IC, Package_SO:TSSOP-8_3x3mm_P0.65mm, symbol local:NT3H2111W0FTTJ
- added LED1: LED, LED_SMD:LED_0805_2012Metric, symbol Device:LED
- added R1: 47Ω, Resistor_SMD:R_0805_2012Metric, symbol Device:R
- added U1: NT3H2111W0FHKH, NT3H2111W0FHKH:QFN8P50_160X160X50L40X20N, symbol NT3H2111W0FKH:NT3H2111W0FHKH
- ANT1: value PCB Antenna -> Class5_Circular_D35mm_ID20mm_8T_W0.56_G0.30; footprint NFC_Antenna:Class4_48x25mm_5T -> Antenna:Class5_Circular_D35mm_ID20mm_8T_W0.56_G0.30; now left out of the parts list
Connections:
- net at ANT1.1: now also U1.1 (LA)
- net at ANT1.2: now also U1.8 (LB)
- net at C1.1: now also R1.2, U1.6 (VCC), U1.7 (VOUT)
- net GND: no longer names the net of C1.2
- net GND: now also LED1.1 (K), U1.2 (VSS)
- new net: LED1.2 (A), R1.1

Commit message: Finalized card's design
Parts:
- removed U1: NT3H2111W0FHKH, NT3H2111W0FHKH:QFN8P50_160X160X50L40X20N, symbol NT3H2111W0FKH:NT3H2111W0FHKH
- added U1: NT3H2111W0FTTJ, Package_SO:TSSOP-8_3x3mm_P0.65mm, symbol NT3H2111W0FKH:NT3H2111W0FTTJ
- LED1: value LED -> LED_Yellow; footprint LED_SMD:LED_0805_2012Metric -> LED_SMD:LED_0603_1608Metric
- R1: value 47Ω -> 1 kΩ
Connections:
- net at ANT1.1: now also U1.1 (LA)
- net at ANT1.2: now also U1.8 (LB)
- net GND: now reaches C1.2, LED1.1 (K)
- net GND: now also U1.2 (VSS)
- net at C1.1, R1.2: now also U1.7 (VOUT)
- no-connect marks 3 -> 4

Commit message: Added production files
Parts:
- C1: LCSC Part # (none) -> C520076
- LED1: value LED_Yellow -> APT1608SYCK/J3-PRV; LCSC Part # (none) -> C5440241
- R1: LCSC Part # (none) -> C17513
- U1: value NT3H2111W0FTTJ -> NT3H2211W0FTTJ; LCSC Part # (none) -> C2654822
Changed lines of the file:
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@@
+			)
+		)
+		(property "LCSC Part #" "C17513"
+			(at 227.33 88.9 0)
+			(hide yes)
+			(show_name no)
+			(do_not_autoplace no)
+			(effects
+				(font
+					(size 1.27 1.27)
+				)
 			)
 		)
@@
 			)
 		)
-		(property "Value" "LED_Yellow"
+		(property "Value" "APT1608SYCK/J3-PRV"
 			(at 231.14 101.9174 90)
 			(hide yes)
@@
 		(property "Sim.Pins" "1=K 2=A"
 			(at 227.33 99.06 0)
+			(hide yes)
+			(show_name no)
+			(do_not_autoplace no)
+			(effects
+				(font
+					(size 1.27 1.27)
+				)
+			)
+		)
+		(property "LCSC Part #" "C5440241"
+			(at 227.33 99.06 90)
 			(hide yes)
 			(show_name no)
@@
 			)
 		)
+		(property "LCSC Part #" "C520076"
+			(at 213.36 90.17 0)
+			(hide yes)
+			(show_name no)
+			(do_not_autoplace no)
+			(effects
+				(font
+					(size 1.27 1.27)
+				)
+			)
+		)
 		(pin "2"
 		)
@@
 			)
 		)
-		(property "Value" "NT3H2111W0FTTJ"
+		(property "Value" "NT3H2211W0FTTJ"
 			(at 170.18 77.47 0)
 			(show_name no)
@@
 			(at 170.18 120.65 0)
 			(hide yes)
+			(show_name no)
+			(do_not_autoplace no)
+			(effects
+				(font
+					(size 1.27 1.27)
+				)
+			)
+		)
+		(property "LCSC Part #" "C2654822"
+			(at 170.18 120.65 0)
+			(hide yes)
